File: LightPipe.kicad_pcb (KiCad board)
At the start: 2 copper layers, 76 x 76 mm, 0 parts

Commit message: first PCB draft
Parts:
- added J1: Conn_01x03, h8-Connectors:Lumberg-KLB-4-Klinkensteckverbinder-3_5, F.Cu at (177.5, 104.3)
- added J2: Conn_01x02, h8-Connectors:XT30, F.Cu at (164.3, 82.7)
- added J3: Conn_01x04, h8-Connectors:APA102-through, B.Cu at (167.6, 98.5)
- added J4: Conn_01x04, h8-Connectors:APA102-through, B.Cu at (173.9, 76.9)
- added J5: Conn_01x04, h8-Connectors:APA102-through, B.Cu at (189.5, 93.1)
- added J6: Conn_01x01, Connector_Wire:SolderWire-0.15sqmm_1x01_D0.5mm_OD1.5mm, B.Cu at (160.5, 90.0)
- added J7: Conn_01x01, Connector_Wire:SolderWire-0.15sqmm_1x01_D0.5mm_OD1.5mm, B.Cu at (164.5, 92.0)
- added J8: Conn_01x02, Connector_PinSocket_2.54mm:PinSocket_1x02_P2.54mm_Vertical, B.Cu at (187.0, 75.6)
- added J9: Conn_01x03, h8-Connectors:Lumberg-KLB-4-Klinkensteckverbinder-3_5, F.Cu at (189.6, 81.7)
Routing:
- net d2: track 0.00 -> 43.0 mm
- net clk2: track 0.00 -> 35.5 mm, vias 0 -> 2
- net GND: track 0.00 -> 24.9 mm, vias 0 -> 2
- net clk1: track 0.00 -> 17.6 mm, vias 0 -> 1
- net d1: track 0.00 -> 11.6 mm, vias 0 -> 1
- net d3: track 0.00 -> 9.78 mm
- net +5V: track 0.00 -> 9.26 mm, vias 0 -> 3
- net clk3: track 0.00 -> 4.56 mm
- added copper zone on F.Cu, net +5V
- added copper zone on B.Cu, net GND
Other:
- board size 76 x 76 mm -> 38.1 x 38.1 mm
- net class Power added: clearance 0.2, trace_width 2, via_dia 1, via_drill 0.5
